File: digital_logic/old_designs/v1_kicad/v1_qiroll PAS digital logic.kicad_pcb (KiCad board)
At the start: 2 copper layers, 53.3 x 45.7 mm, 43 parts, among them J1 led_sw1, J2 mode_thr_batt, J3 pas_sense, J4 brk_sense, J5 jumper, U1 14538, U2 4023, U3 4027, U4 14538, U5 L7805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

Commit message: pcb revision, add circuit sim, old kicad files to reference for v1 board repairs
Parts:
- removed D1: Reverse Protect Diode, Diode_SMD:D_MiniMELF
- removed F1: PTC, Fuse:Fuse_1206_3216Metric
- removed R11: 10k, Resistor_SMD:R_0603_1608Metric
- C11: value .1u -> 1u
- moved R10 4.46 mm to (118.7, 56.5)
- moved C10 2.03 mm to (117.5, 78.1)
Connections:
- J2 pad 2: Net-(F1-Pad2) -> Net-(J2-Pad2)
- R10 pad 2: Net-(D1-Pad1) -> Net-(J2-Pad2)
- U6 pad 6: VCC -> Net-(U2-Pad1)
Routing:
- net Net-(D1-Pad1): track 28.4 -> 0.00 mm
- net VCC: track 270.2 -> 241.8 mm
- net Net-(U2-Pad1): track 13.7 -> 39.5 mm, vias 2 -> 4
- net GND: track 70.0 -> 74.6 mm, vias 17 -> 18
- net Net-(F1-Pad2): track 4.35 -> 0.00 mm
- net BRK: track 60.5 -> 57.0 mm
- net Net-(J2-Pad2): track 0.00 -> 3.25 mm
- net Net-(J3-Pad3): track 46.1 -> 43.3 mm
- net Net-(C10-Pad1): track 11.1 -> 13.2 mm
- net Net-(C10-Pad2): track 19.9 -> 21.8 mm
- net Net-(U1-Pad10): track 56.5 -> 54.9 mm
- net Net-(J2-Pad4): track 24.2 -> 23.5 mm
- net Net-(C6-Pad1): track 15.9 -> 16.6 mm
Other:
- board text added: "qiroll pedal assist v1 Eric Dasmalchi"
- board text removed: "qiroll pedal assist v1.1 Eric Dasmalchi"

Commit message: add old design safety notes, delete faulty gerbers
Connections:
- U6 pad 6: Net-(U2-Pad1) -> VCC
Routing:
- net Net-(U2-Pad1): track 39.5 -> 13.7 mm, vias 4 -> 2
- net VCC: track 241.8 -> 256.6 mm
Changed lines of the file:
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@@
     (thickness 1.6)
     (drawings 18)
-    (tracks 604)
+    (tracks 597)
     (zones 0)
     (modules 40)
@@
   (layers
     (0 F.Cu signal)
-    (31 B.Cu signal hide)
+    (31 B.Cu signal)
     (33 F.Adhes user)
     (35 F.Paste user)
@@
       (net 1 GND))
     (pad 6 smd roundrect (at -2.475 2.54 270) (size 1.95 0.6) (layers F.Cu F.Paste F.Mask) (roundrect_rratio 0.25)
-      (net 29 "Net-(U2-Pad1)"))
+      (net 22 VCC))
     (pad 5 smd roundrect (at -2.475 1.27 270) (size 1.95 0.6) (layers F.Cu F.Paste F.Mask) (roundrect_rratio 0.25)
       (net 25 "Net-(C11-Pad2)"))
@@
   (segment (start 139.192 69.596) (end 137.450999 67.854999) (width 0.25) (layer B.Cu) (net 22))
   (segment (start 144.054999 65.749001) (end 146.812 62.992) (width 0.25) (layer B.Cu) (net 22))
+  (segment (start 145.42499 55.23501) (end 147.32 53.34) (width 0.25) (layer F.Cu) (net 22))
+  (segment (start 144.112001 62.701001) (end 145.42499 61.388012) (width 0.25) (layer F.Cu) (net 22))
+  (segment (start 143.415999 62.701001) (end 144.112001 62.701001) (width 0.25) (layer F.Cu) (net 22))
+  (segment (start 145.42499 61.388012) (end 145.42499 55.23501) (width 0.25) (layer F.Cu) (net 22))
+  (segment (start 142.24 61.525002) (end 143.415999 62.701001) (width 0.25) (layer F.Cu) (net 22))
+  (segment (start 142.24 59.755) (end 142.24 61.525002) (width 0.25) (layer F.Cu) (net 22))
   (segment (start 116.65 78.155) (end 116.7 78.105) (width 0.25) (layer F.Cu) (net 23))
   (segment (start 116.65 82.55) (end 116.65 78.155) (width 0.25) (layer F.Cu) (net 23))
@@
   (segment (start 130.20999 75.218242) (end 130.20999 76.50999) (width 0.25) (layer F.Cu) (net 28))
   (segment (start 131 74.93) (end 130.498232 74.93) (width 0.25) (layer F.Cu) (net 28))
-  (via (at 133.604 77.216) (size 0.8) (drill 0.4) (layers F.Cu B.Cu) (net 29))
   (via (at 129.54 80.01) (size 0.8) (drill 0.4) (layers F.Cu B.Cu) (net 29))
   (via (at 129.54 83.185) (size 0.8) (drill 0.4) (layers F.Cu B.Cu) (net 29))
@@
   (segment (start 129.54 79.444315) (end 130.879315 78.105) (width 0.25) (layer F.Cu) (net 29))
   (segment (start 129.54 80.01) (end 129.54 79.444315) (width 0.25) (layer F.Cu) (net 29))
-  (via (at 142.24 61.976) (size 0.8) (drill 0.4) (layers F.Cu B.Cu) (net 29))
-  (segment (start 132.715 78.105) (end 131.51 78.105) (width 0.25) (layer F.Cu) (net 29))
-  (segment (start 133.604 77.216) (end 132.715 78.105) (width 0.25) (layer F.Cu) (net 29))
-  (segment (start 142.24 61.976) (end 142.24 59.755) (width 0.25) (layer F.Cu) (net 29))
-  (segment (start 138.684 61.976) (end 142.24 61.976) (width 0.25) (layer B.Cu) (net 29))
-  (segment (start 137.72599 62.93401) (end 138.684 61.976) (width 0.25) (layer B.Cu) (net 29))
-  (segment (start 134.112 67.564) (end 137.72599 63.95001) (width 0.25) (layer B.Cu) (net 29))
-  (segment (start 134.112 74.618998) (end 134.112 67.564) (width 0.25) (layer B.Cu) (net 29))
-  (segment (start 133.386999 75.343999) (end 134.112 74.618998) (width 0.25) (layer B.Cu) (net 29))
-  (segment (start 133.386999 76.998999) (end 133.386999 75.343999) (width 0.25) (layer B.Cu) (net 29))
-  (segment (start 137.72599 63.95001) (end 137.72599 62.93401) (width 0.25) (layer B.Cu) (net 29))
-  (segment (start 133.604 77.216) (end 133.386999 76.998999) (width 0.25) (layer B.Cu) (net 29))
   (via (at 136.144 71.628) (size 0.8) (drill 0.4) (layers F.Cu B.Cu) (net 30))
   (via (at 141.732 73.152) (size 0.8) (drill 0.4) (layers F.Cu B.Cu) (net 30))
@@
     (polygon
       (pts
-        (xy 149.86 73.66) (xy 134.112 73.66) (xy 134.112 68.072) (xy 149.86 68.072)
-      )
-    )
-  )
-  (zone (net 0) (net_name "") (layer B.Cu) (hatch edge 0.508)
-    (connect_pads (clearance 0.508))
-    (min_thickness 0.254)
-    (keepout (tracks allowed) (vias allowed) (copperpour not_allowed))
-    (fill (arc_segments 32) (thermal_gap 0.508) (thermal_bridge_width 0.508))
-    (polygon
-      (pts
         (xy 143.764 72.8345) (xy 143.764 78.5495) (xy 138.176 78.586973) (xy 138.176 72.871973)
       )
@@
       )
     )
+  )
+  (zone (net 0) (net_name "") (layer B.Cu) (hatch edge 0.508)
+    (connect_pads (clearance 0.508))
+    (min_thickness 0.254)
+    (keepout (tracks allowed) (vias allowed) (copperpour not_allowed))
+    (fill (arc_segments 32) (thermal_gap 0.508) (thermal_bridge_width 0.508))
+    (polygon
+      (pts
+        (xy 149.86 73.66) (xy 134.112 73.66) (xy 134.112 68.072) (xy 149.86 68.072)
+      )
+    )
