File: digital_logic_build/kicad/qiroll PAS digital logic.sch (KiCad schematic (older format))
At the start: 47 parts, among them J1 brk_sense, J2 led_sw1, J4 mode_thr_batt, J5 pas_sense, U1 4093B, U2 4027B, U3 4093B, U5 4093B, U6 14538B, U7 L78L05_TO92

Commit message: version 2.5
Parts:
- removed J1: brk_sense, Connector_PinHeader_2.54mm:PinHeader_1x02_P2.54mm_Vertical, symbol Connector:Conn_01x02_Male
- added J5: 3_pin, Connector_PinHeader_2.54mm:PinHeader_1x03_P2.54mm_Vertical, symbol Connector:Conn_01x03_Male
- J2: footprint Connector_PinHeader_2.54mm:PinHeader_1x03_P2.54mm_Vertical -> Connector_PinHeader_2.54mm:PinHeader_1x04_P2.54mm_Vertical; symbol Connector:Conn_01x03_Male -> Connector:Conn_01x04_Male
- J3: renamed from J5; value pas_sense -> accessory
- R2: value 1.6k -> 75k
- R7: value 1.6k -> 3.3k
- U7: value L78L05_TO92 -> MCP1799_3V3; footprint Package_TO_SOT_THT:TO-92_Inline -> Package_TO_SOT_SMD:SOT-23; symbol Regulator_Linear:L78L05_TO92 -> Regulator_Linear:MCP1700-3302E_SOT23
Connections:
- net GND: now also U7.1 (GND), J5.2 (Pin_2); no longer U7.2 (GND)
- net VDD: now also U7.2 (VO); no longer U7.1 (VO)
- net at C2.2, R3.2, U3.8: now also J2.3 (Pin_3); no longer J2.2 (Pin_2)
- net at U3.3: now also J2.4 (Pin_4); no longer J2.3 (Pin_3)
- net at F1.2, J4.2 (Pin_2): now also J5.3 (Pin_3)
- net at D2.1 (K), R2.2, U3.6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: now also J2.2 (Pin_2), J5.1 (Pin_1)
Other:
- note added: "LED (1.5ma max!)"
- note added: "LED Behavior:\npedal assist on, regen off: solid on\npedal assist on, regen on (or actively braking): flashes\npedal assist off, regen off: off\npedal assist off, regen on (or actively braking): flashes"
- note added: "accessory_gnd"
- note added: "accessory_pwr"
- note added: "battery input PTC protection\n3.3v linear regulator\nmin current approx. 225ua\nmax current approx. 3ma"
- note added: "brake_in"
- note added: "brake_out"
- note added: "don’t install D2 for std"
- note added: "don’t install\nD5 for std"
- note added: "regen on/off FF, double-click toggles, \nreset on pedaling"
- note added: "rgn brk/mode\n(low=on)"
- note removed: "LED"
- note removed: "LED Behavior:\npedal assist on, regen off: solid on\npedal assist on, regen on: flashes\npedal assist off, regen off: off\npedal assist off, regen on: flashes"
- note removed: "battery input PTC protection\n5v linear regulator (input max 20v or 33v after R7 drop)\nmin current approx. 3ma\nmax current approx. 5ma"
- note removed: "brake"
- note removed: "regen braking/mode\n(low=on)"
- note removed: "regen on/off FF, double-click toggles, \nreset on pedaling, set on braking"
- moved on the sheet: C1, C2, C3, C8, C9, D2, D3, D4, D5, JP1, R1, R10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
